Commit message: minor changes in urdf

File: urdf/rover.urdf (robot description, URDF)
Before this commit: robot rover, 8 links, 7 joints
Links:
- added link base_link
Joints:
- added joint chassis_joint: type fixed, parent base_link, child chassis, origin xyz=0.0 0.0 0.0 rpy=0.0 0.0 0.0
- joint lidar_mount_joint: axis 0.0 0.0 1.0 -> (none)
